File: Hardware/Payload URC/MCU_interface_vibrator.kicad_sch (KiCad schematic)
At the start: 2 parts

Commit message: Testing github skill issue
Parts:
- R46, R47: value 4.7kΩ -> 4.7k
Changed lines of the file:
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@@
 			)
 		)
-		(property "Value" "4.7kΩ"
+		(property "Value" "4.7k"
 			(at 133.35 101.5999 0)
 			(show_name no)
@@
 			)
 		)
-		(property "Value" "4.7kΩ"
+		(property "Value" "4.7k"
 			(at 115.57 81.2799 0)
 			(show_name no)
