File: Hardware/Payload URC/Main_Board_Communication.kicad_sch (KiCad schematic)
At the start: 6 parts, among them J5 Conn_01x03, U10 THVD1500DR, U8 TPD4E05U06DQAR

Commit message: Testing github skill issue
Parts:
- C17: value 0.1uF -> 0.1u; Voltage Voltage -> 25V
- R21: value 120Ω -> 120
- R40: value 10kΩ -> 10k
Changed lines of the file:
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@@
 			)
 		)
-		(property "Value" "120Ω"
+		(property "Value" "120"
 			(at 146.05 88.8999 0)
 			(show_name no)
@@
 			)
 		)
-		(property "Value" "0.1uF"
+		(property "Value" "0.1u"
 			(at 166.37 89.7115 0)
 			(show_name no)
@@
 			)
 		)
-		(property "Voltage" "Voltage"
+		(property "Voltage" "25V"
 			(at 166.37 92.2515 0)
 			(show_name no)
@@
 			)
 		)
-		(property "Value" "10kΩ"
+		(property "Value" "10k"
 			(at 83.82 102.8699 0)
 			(show_name no)
