File: Hardware/Payload URC/PAYLOAD-URC.kicad_pcb (KiCad board)
At the start: 4 copper layers, 0 parts

Commit message: Updated files
Parts:
- added C1: 1u, SCRB_STD_Passives:C0805, F.Cu at (45.2, 77.5)
- added C10: 12p, SCRB_STD_Passives:C0805, F.Cu at (70.6, 77.0)
- added C11: 2.2u, SCRB_STD_Passives:C0805, F.Cu at (60.0, 70.0)
- added C13: 12p, SCRB_STD_Passives:C0805, F.Cu at (56.5, 83.0)
- added C17: 0.1u, SCRB_STD_Passives:C0805, F.Cu at (60.0, 104.0)
- added C18: 0.1u, SCRB_STD_Passives:C0805, F.Cu at (77.0, 100.0)
- added C19: 4.2p, SCRB_STD_Passives:C0805, F.Cu at (77.0, 104.5)
- added C2: 1u, SCRB_STD_Passives:C0805, F.Cu at (76.3, 73.8)
- added C20: 1u, SCRB_STD_Passives:C0805, F.Cu at (62.5, 97.0)
- added C21: 1u, SCRB_STD_Passives:C0805, F.Cu at (62.5, 101.5)
- added C22: 2.2u, SCRB_STD_Passives:C0805, F.Cu at (79.5, 73.5)
- added C26: 0.1u, SCRB_STD_Passives:C0805, F.Cu at (70.5, 82.0)
- added C3: 0.1u, SCRB_STD_Passives:C0402, F.Cu at (73.5, 72.3)
- added C4: 0.1u, SCRB_STD_Passives:C0805, F.Cu at (70.6, 80.0)
- added C5: 1u, SCRB_STD_Passives:C0805, F.Cu at (51.5, 69.5)
- added C6: 0.1u, SCRB_STD_Passives:C0402, F.Cu at (73.5, 73.9)
- added C7: 0.1u, SCRB_STD_Passives:C0402, F.Cu at (73.5, 75.5)
- added C8: 4.7u, SCRB_STD_Passives:C0603, F.Cu at (73.5, 70.3)
- added D3: TVS_SOD523, SCRB_STD_Actives:SOD-523, F.Cu at (54.5, 95.1)
- added D4: BPW34, OptoDevice:Osram_DIL2_4.3x4.65mm_P5.08mm, F.Cu at (77.5, 109.5)
- added D8: 1N5819, Diode_THT:D_DO-41_SOD81_P10.16mm_Horizontal, F.Cu at (103.5, 96.3)
- added D9: 1N5819, Diode_THT:D_DO-41_SOD81_P10.16mm_Horizontal, F.Cu at (89.5, 99.0)
- added H1: MountingHole, MountingHole:MountingHole_3mm_Pad_TopBottom, F.Cu at (37.5, 66.5)
- added H2: MountingHole, MountingHole:MountingHole_3mm_Pad_TopBottom, F.Cu at (117.5, 66.0)
- added H3: MountingHole, MountingHole:MountingHole_3mm_Pad_TopBottom, F.Cu at (117.5, 112.5)
- added H4: MountingHole, MountingHole:MountingHole_3mm_Pad_TopBottom, F.Cu at (37.5, 113.0)
- added J1: VG2080001H, SCRB_Connectors:JST-GH-SM04B-GHS-TB, F.Cu at (66.0, 108.5)
- added J18: Conn_01x02, SCRB_Connectors:JST-GH-SM04B-GHS-TB, F.Cu at (95.9, 110.5)
- added J2: Conn_01x02, Connector_JST:JST_PH_S2B-PH-K_1x02_P2.00mm_Horizontal, F.Cu at (109.2, 76.7)
- added J20: Conn_01x02, SCRB_Connectors:JST-GH-SM04B-GHS-TB, F.Cu at (105.9, 110.7)
- added J3: Conn_01x02, Connector_JST:JST_PH_S2B-PH-K_1x02_P2.00mm_Horizontal, F.Cu at (109.0, 84.5)
- added J4: Conn_01x02, Connector_Molex:Molex_Micro-Fit_3.0_43650-0215_1x02_P3.00mm_Vertical, F.Cu at (44.2, 71.0)
- added J5: Conn_01x03, Connector_Hirose:Hirose_DF57H-3P-1.2V_1x03_P1.2mm_Socket, F.Cu at (45.0, 106.5)
- added J6: ST-Link-Conn-SM, Connector_JST:JST_PH_B4B-PH-SM4-TB_1x04-1MP_P2.00mm_Vertical, F.Cu at (46.5, 96.0)
- added J7: Conn_01x02, Connector_Molex:Molex_Micro-Fit_3.0_43650-0215_1x02_P3.00mm_Vertical, F.Cu at (44.2, 83.0)
- added J8: Conn_01x03, Connector_Hirose:Hirose_DF57H-3P-1.2V_1x03_P1.2mm_Socket, F.Cu at (72.8, 109.4)
- added LD1: LED0603, SCRB_STD_Actives:LED0603, F.Cu at (81.5, 86.8)
- added LD2: LED0603, SCRB_STD_Actives:LED0603, F.Cu at (83.5, 86.8)
- added LD3: LED0603, SCRB_STD_Actives:LED0603, F.Cu at (63.3, 72.5)
- added LD4: LED0603, SCRB_STD_Actives:LED0603, F.Cu at (63.3, 70.0)
- added Q1: AO3400A, Package_TO_SOT_SMD:SOT-23, F.Cu at (90.0, 93.6)
- added Q2: AO3400A, Package_TO_SOT_SMD:SOT-23, F.Cu at (97.0, 93.0)
- added Q5: AO3400A, Package_TO_SOT_SMD:SOT-23, F.Cu at (98.9, 78.0)
- added Q6: AO3400A, Package_TO_SOT_SMD:SOT-23, F.Cu at (98.9, 85.0)
- added R1: 10k, SCRB_STD_Passives:R0402, F.Cu at (81.3, 83.8)
- added R11: 4.7k, SCRB_STD_Passives:R0805, F.Cu at (79.5, 70.5)
- added R17: 10k, SCRB_STD_Passives:R0805, F.Cu at (79.6, 72.0)
- added R2: 10k, SCRB_STD_Passives:R0402, F.Cu at (83.0, 83.8)
- added R20: 100, SCRB_STD_Passives:R0805, F.Cu at (76.0, 86.0)
- added R21: 120, SCRB_STD_Passives:R0805, F.Cu at (59.9, 106.0)
- added R24: 100, SCRB_STD_Passives:R0805, F.Cu at (88.4, 78.5)
- added R28: 10, SCRB_STD_Passives:R0805, F.Cu at (98.4, 100.5)
- added R29: 10, SCRB_STD_Passives:R0805, F.Cu at (98.5, 99.0)
- added R3: 10k, SCRB_STD_Passives:R0402, F.Cu at (59.5, 72.5)
- added R30: 10k, SCRB_STD_Passives:R0805, F.Cu at (79.0, 87.5)
- added R31: 10k, SCRB_STD_Passives:R0805, F.Cu at (76.0, 87.5)
- added R32: 100, SCRB_STD_Passives:R0805, F.Cu at (79.0, 86.0)
- added R33: 100, SCRB_STD_Passives:R0805, F.Cu at (87.9, 70.5)
- added R34: 10k, SCRB_STD_Passives:R0805, F.Cu at (88.0, 72.0)
- added R35: 10k, SCRB_STD_Passives:R0805, F.Cu at (88.4, 80.0)
- added R36: 100, SCRB_STD_Passives:R0805, F.Cu at (104.0, 76.5)
- added R37: 100, SCRB_STD_Passives:R0805, F.Cu at (104.4, 84.0)
- added R4: 10k, SCRB_STD_Passives:R0402, F.Cu at (59.5, 71.5)
- added R40: 10k, SCRB_STD_Passives:R0805, F.Cu at (49.4, 106.0)
- added R41: 2.2k, SCRB_STD_Passives:R0805, F.Cu at (84.4, 78.8)
- added R42: 2.2k, SCRB_STD_Passives:R0805, F.Cu at (84.4, 80.2)
- added R43: 4.7k, SCRB_STD_Passives:R0805, F.Cu at (84.4, 81.8)
- added R44: 1M, SCRB_STD_Passives:R0805, F.Cu at (78.5, 104.5)
- added R45: 6.6k, SCRB_STD_Passives:R0805, F.Cu at (78.5, 99.9)
- added R46: 4.7k, SCRB_STD_Passives:R0805, F.Cu at (84.4, 74.3)
- added R47: 4.7k, SCRB_STD_Passives:R0805, F.Cu at (84.4, 76.8)
- added R8: 4.7k, SCRB_STD_Passives:R0805, F.Cu at (79.5, 69.0)
- added SW2: SW_Oval, SCRB_Electromechanical:SW_C2888430, F.Cu at (64.6, 88.9)
- added TP10: TestPoint, TestPoint:TestPoint_Loop_D2.60mm_Drill1.6mm_Beaded, F.Cu at (88.5, 88.5)
- added TP12: TestPoint, TestPoint:TestPoint_Loop_D2.60mm_Drill1.6mm_Beaded, F.Cu at (92.5, 88.5)
- added TP14: TestPoint, TestPoint:TestPoint_Loop_D2.60mm_Drill1.6mm_Beaded, F.Cu at (95.0, 77.5)
- added TP16: TestPoint, TestPoint:TestPoint_Loop_D2.60mm_Drill1.6mm_Beaded, F.Cu at (94.5, 84.0)
- added TP18: TestPoint, TestPoint:TestPoint_Loop_D2.60mm_Drill1.6mm_Beaded, F.Cu at (73.5, 95.5)
- added TP19: TestPoint, TestPoint:TestPoint_Loop_D2.60mm_Drill1.6mm_Beaded, F.Cu at (78.0, 95.5)
- added TP2: TestPoint, TestPoint:TestPoint_Loop_D2.60mm_Drill1.6mm_Beaded, F.Cu at (62.0, 79.0)
- added TP20: TestPoint, TestPoint:TestPoint_Loop_D2.60mm_Drill1.6mm_Beaded, F.Cu at (82.5, 95.5)
- added TP21: TestPoint, TestPoint:TestPoint_Loop_D2.60mm_Drill1.6mm_Beaded, F.Cu at (82.0, 100.0)
- added TP26: TestPoint, TestPoint:TestPoint_Loop_D2.60mm_Drill1.6mm_Beaded, F.Cu at (82.0, 104.5)
- added TP35: TestPoint, TestPoint:TestPoint_Loop_D2.60mm_Drill1.6mm_Beaded, F.Cu at (61.0, 93.5)
- added TP36: TestPoint, TestPoint:TestPoint_Loop_D2.60mm_Drill1.6mm_Beaded, F.Cu at (65.0, 93.5)
- added TP37: TestPoint, TestPoint:TestPoint_Loop_D2.60mm_Drill1.6mm_Beaded, F.Cu at (69.0, 93.5)
- added U10: THVD1500DR, SCRB_TexasInstruments:D0008A, F.Cu at (54.5, 106.5)
- added U3: TPD4E05U06DQAR, SCRB_TexasInstruments:DQA0010A, F.Cu at (53.4, 102.6)
- added U4: TLV75533PDBV, Package_TO_SOT_SMD:SOT-23-5, F.Cu at (52.6, 82.0)
- added U5: ADS1115IDGS, Package_SO:TSSOP-10_3x3mm_P0.5mm, F.Cu at (73.0, 100.7)
- added U6: STM32C542CCT6, SCRB_Misc_ICs:LQFP-48_7x7mm_P0.5mm, F.Cu at (77.5, 79.5)
- added U8: TPD4E05U06DQAR, SCRB_TexasInstruments:DQA0010A, F.Cu at (59.4, 108.5)
- added U9: TPS7A20xxxDBV, Package_TO_SOT_SMD:SOT-23-5, F.Cu at (55.4, 71.0)
- added Y1: XTAL3225 (16M, 9P), SCRB_STD_Passives:SMD3225, F.Cu at (64.3, 84.4)
Routing:
- net GND: vias 0 -> 2
- net /3V3: vias 0 -> 4
- net (no net): vias 0 -> 1
- added copper zone on In2.Cu, net /3V3
- added copper zone on In1.Cu, net GND
Other:
- board outline added: 87 x 54 mm
- board text added: "SSS"
- board text added: "Surface Analysis System 405nm, 445nm, ADC, Vibrator"

Commit message: Update
Parts:
- removed C17: 0.1u, SCRB_STD_Passives:C0805
- removed J18: Conn_01x02, SCRB_Connectors:JST-GH-SM04B-GHS-TB
- removed J5: Conn_01x03, Connector_Hirose:Hirose_DF57H-3P-1.2V_1x03_P1.2mm_Socket
- removed R21: 120, SCRB_STD_Passives:R0805
- removed R28, R29: 10, SCRB_STD_Passives:R0805
- removed R40: 10k, SCRB_STD_Passives:R0805
- removed R45: 6.6k, SCRB_STD_Passives:R0805
- removed TP19, TP20, TP26, TP36, TP37: TestPoint, TestPoint:TestPoint_Loop_D2.60mm_Drill1.6mm_Beaded
- removed U10: THVD1500DR, SCRB_TexasInstruments:D0008A
- removed U8: TPD4E05U06DQAR, SCRB_TexasInstruments:DQA0010A
- added J19: Conn_01x02, SCRB_Connectors:JST-GH-SM04B-GHS-TB, F.Cu at (83.2, 105.2)
- added J9: Conn_01x03, Connector_Hirose:Hirose_DF57H-3P-1.2V_1x03_P1.2mm_Socket, F.Cu at (69.0, 105.6)
- added R22: 120, SCRB_STD_Passives:R0805, F.Cu at (62.5, 106.7)
- added U1: DRV2605LDGS, Package_SO:TSSOP-10_3x3mm_P0.5mm, F.Cu at (101.2, 98.0)
- added U11: THVD1500DR, SCRB_TexasInstruments:D0008A, F.Cu at (58.0, 106.2)
- C19: value 4.2p -> 0.1u
- D4: value BPW34 -> TVS_SOD523; footprint OptoDevice:Osram_DIL2_4.3x4.65mm_P5.08mm -> SCRB_STD_Actives:SOD-523
- H1, H2, H3, H4: value MountingHole -> MH2.5
- R44: value 1M -> 10k
- moved J1 43.1 mm to (107.8, 98.3), turned to 90 degrees
- moved C20 40.1 mm to (102.5, 93.8), turned to 180 degrees
- moved U9 39.1 mm to (90.5, 88.2), turned to 180 degrees
- moved C21 38.8 mm to (101.2, 102.5), turned to 0 degrees
- moved TP35 36.5 mm to (97.5, 94.5)
- moved C11 33.4 mm to (87.6, 88.8), turned to 90 degrees
- moved R4 32.0 mm to (86.1, 89.3), turned to 90 degrees
- moved LD4 29.0 mm to (84.6, 89.6), turned to 90 degrees
- moved R44 25.1 mm to (53.5, 106.2), turned to 90 degrees
- moved J8 24.0 mm to (49.1, 105.1), turned to 180 degrees
- moved D4 21.0 mm to (83.1, 89.3), turned to -90 degrees
- moved D8 20.6 mm to (100.0, 76.1), turned to 90 degrees
- moved C2 18.2 mm to (60.7, 83.0), turned to -90 degrees
- moved TP2 17.1 mm to (51.5, 92.5)
- moved D3 16.8 mm to (65.2, 82.2), turned to 90 degrees
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Connections:
- C19 pad 1: Net-(D4-K) -> /5V
- C19 pad 2: Net-(C19-Pad2) -> GND
- D4 pad 1: Net-(D4-K) -> GND
- D4 pad 2: GND -> /4V
- J8 pad 1: Net-(J8-Pin_1) -> /JTCK/SWCLK
- J8 pad 2: Net-(J8-Pin_2) -> /ESD_protection/RS485A
- R44 pad 1: Net-(D4-K) -> GND
- R44 pad 2: Net-(C19-Pad2) -> Net-(U11-DE)
- U3 pad 4: unconnected-(U3-D3-Pad4) -> /ESD_protection/RS485A
- U3 pad 7: unconnected-(U3-NC-Pad7) -> /ESD_protection/RS485A
- U3 pad 9: unconnected-(U3-NC-Pad9) -> /JTCK/SWCLK
Routing:
- net GND: track 0.00 -> 57.9 mm, vias 2 -> 86
- net /3V3: track 0.00 -> 34.3 mm, vias 4 -> 9
- net /5V: track 0.00 -> 15.0 mm, vias 0 -> 2
- net /4V: track 0.00 -> 9.38 mm, vias 0 -> 3
- net /12V: track 0.00 -> 7.16 mm, vias 0 -> 3
- net /I2C1_SDA: track 0.00 -> 2.98 mm
- net /I2C1_SCL: track 0.00 -> 2.24 mm
- net /GPIO: track 0.00 -> 2.03 mm
- net /UART4_TX: track 0.00 -> 1.85 mm
- net Net-(LD4-A): track 0.00 -> 1.50 mm
- net /I2C1_SCL_1: track 0.00 -> 1.46 mm
- net /I2C1_SDA_1: track 0.00 -> 0.74 mm
- net /PB14_GPIO: track 0.00 -> 0.68 mm
- added copper zone on In2.Cu, net /12V
- added copper zone on In2.Cu, net /4V
- added copper zone on In2.Cu, net /5V
- added copper zone on B.Cu, net GND
Other:
- board size 87 x 54 mm -> 75 x 49 mm
- board text added: "12V"
- board text added: "12V here"
- board text added: "3V3"
- board text added: "3V3 here"
- board text added: "405 nm 445 nm LEDs"
- board text added: "4V"
- board text added: "4V here"
- board text added: "5V"
- board text added: "ADC Converter"
- board text added: "Driver"
- board text added: "FHS"
- board text added: "Flyback diodes"
- board text added: "MCU Communication"
- board text added: "MOSFETs"
- board text added: "Photodiode"
- board text added: "SAS 405nm 445 nm + Photodiode"
- board text added: "SSS Vibrator"
- board text added: "STI-LINK PORT"
- board text added: "Solenoids"
- board text added: "Vibrator"
- board text removed: "SSS"
- board text removed: "Surface Analysis System 405nm, 445nm, ADC, Vibrator"
