File: Hardware/Payload URC/PAYLOAD-URC.kicad_sch (KiCad schematic)
At the start: 23 parts, among them J8 Conn_01x04, J9 Conn_01x04, SW1 SW_Push, U4 TLV75533PDBV, U6 STM32C542CCT6, U9 TPS7A20xxxDBV, Y1 XTAL3225 (16M, 9P)

Commit message: Testing github skill issue
Parts:
- removed C12: 4.7uF, SCRB_STD_Passives:C0805, symbol SCRB_STD_Passives:C0805
- removed C23: 0.1unF, SCRB_STD_Passives:C0805, symbol SCRB_STD_Passives:C0805
- removed C24, C25: 0.1uF, SCRB_STD_Passives:C0805, symbol SCRB_STD_Passives:C0805
- removed J8, J9: Conn_01x04, Connector_Phoenix_MC:PhoenixContact_MCV_1,5_4-G-3.5_1x04_P3.50mm_Vertical, symbol Connector_Generic:Conn_01x04
- removed SW1: SW_Push, symbol Switch:SW_Push
- added C3, C6, C7: 0.1u, SCRB_STD_Passives:C0402, symbol SCRB_STD_Passives:C0402
- added C8: 4.7u, SCRB_STD_Passives:C0603, symbol SCRB_STD_Passives:C0603
- added D3: TVS_SOD523, SCRB_STD_Actives:SOD-523, symbol SCRB_STD_Actives:TVS_SOD523
- added J4, J7: Conn_01x02, Connector_JST:JST_XH_B2B-XH-A_1x02_P2.50mm_Vertical, symbol Connector_Generic:Conn_01x02
- added LD3, LD4: LED0603, SCRB_STD_Actives:LED0603, symbol SCRB_STD_Actives:LED0603
- added R3, R4: 10k, SCRB_STD_Passives:R0402, symbol SCRB_STD_Passives:R0402
- added SW2: SW_Oval, SCRB_Electromechanical:SW_C2888430, symbol SCRB_Electromechanical:SW_Oval
- C1, C2: value 1uF -> 1u; Voltage Voltage -> 25V
- C10, C13: Voltage Voltage -> 25V
- C11: value 2.2μF -> 2.2u; Voltage Voltage -> 25V
- C22: value 2.2uF -> 2.2u; Voltage Voltage -> 25V
- C26: value 0.1uF -> 0.1u; Voltage Voltage -> 25V
- C4: value 0.1μF -> 0.1u; Voltage Voltage -> 25V
- C5: value 1μF -> 1u; Voltage Voltage -> 25V
Connections:
- net 12V: now also C5.1, U9.1 (IN), U9.3 (EN), J4.1 (Pin_1)
- net 3V3: now also C3.1, C6.1, C7.1, C8.1, D3.2 (A2), R3.1
- net 4V: now also R4.1
- net 5V: now also C1.1, U4.1 (IN), J7.1 (Pin_1)
- net GND: now also C3.2, C6.2, C7.2, C8.2, D3.1 (A1), J4.2 (Pin_2), J7.2 (Pin_2), LD3.1 (K), LD4.1 (K), SW2.1; no longer C1.1, U4.1 (IN)
- net NRST: now also SW2.2
- new net: LD4.2 (A), R4.2
- new net: LD3.2 (A), R3.2
- no-connect marks 3 -> 1
Other:
- note added: "Assertions and verifications"
- note added: "FHS solenoids"
- note added: "Notes from meetings"
- note added: "Pre-mask buffer stm32 chip check"
- note added: "Sub boards 3cmx3cm layout mounting holes greater than >2.5mm"
- note added: "Vertical connectors only here"

Commit message: Testing 2
Parts:
- C10, C13: value 12pF -> 12p
Changed lines of the file:
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@@
 			)
 		)
-		(property "Value" "12pF"
+		(property "Value" "12p"
 			(at 225.6016 166.37 90)
 			(show_name no)
@@
 			)
 		)
-		(property "Value" "12pF"
+		(property "Value" "12p"
 			(at 225.6016 189.23 90)
 			(show_name no)

Commit message: Updated files
Parts:
- added H1, H2, H3, H4: MountingHole, MountingHole:MountingHole_3mm_Pad_TopBottom, symbol Mechanical:MountingHole
- J4, J7: footprint Connector_JST:JST_XH_B2B-XH-A_1x02_P2.50mm_Vertical -> Connector_Molex:Molex_Micro-Fit_3.0_43650-0215_1x02_P3.00mm_Vertical
Other:
- note added: "Change mounting holes to =2.5"
- note added: "Daisy chain or chain linked technical report noise consideration wednesday"
- note added: "JST PH or HX for connectors to extension boards"
- note added: "bolts on the middle of the board or diagonals for mounting"

Commit message: Update
Parts:
- added D4: TVS_SOD523, SCRB_STD_Actives:SOD-523, symbol SCRB_STD_Actives:TVS_SOD523
- H1, H2, H3, H4: value MountingHole -> MH2.5; KiLib_Generator (none) -> mounting_hardware/mounting_hole
- J4, J7: KiLib_Generator (none) -> connector/Molex
- U4, U9: KiLib_Generator (none) -> package/gullwing
Connections:
- net 4V: now also D4.2 (A2)
- net GND: now also D4.1 (A1)
Other:
- removed sheet MCU_communication
- sheet ESD_protection ports: added 5V, USART6_RX, USART6_TX; removed none
- moved on the sheet: H1, H2, H3, H4, R11, R8
