File: Hardware/Payload URC/esd.kicad_sch (KiCad schematic)
At the start: 3 parts, among them J6 ST-Link-Conn-SM, U3 TPD4E05U06DQAR

Commit message: Testing github skill issue
Connections:
- net JTDO-SWO: no longer names the net of U3.4 (D3)
- net NRST: no longer names the net of U3.5 (D4)
- no-connect marks 4 -> 6
Changed lines of the file:
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@@
 		(at 167.64 54.61)
 	)
-	(wire
-		(pts
-			(xy 124.46 64.77) (xy 137.16 64.77)
-		)
-		(stroke
-			(width 0)
-			(type default)
-		)
+	(no_connect
+		(at 137.16 69.85)
+	)
+	(no_connect
+		(at 137.16 64.77)
 	)
 	(wire
@@
 	(wire
 		(pts
-			(xy 124.46 69.85) (xy 137.16 69.85)
-		)
-		(stroke
-			(width 0)
-			(type default)
-		)
-	)
-	(wire
-		(pts
 			(xy 123.19 54.61) (xy 137.16 54.61)
 		)
@@
 		)
 	)
-	(hierarchical_label "NRST"
-		(shape input)
-		(at 81.28 83.82 0)
-		(effects
-			(font
-				(size 1.27 1.27)
-			)
-			(justify left)
-		)
-	)
 	(hierarchical_label "JTCK-SWCLK"
 		(shape input)
 		(at 80.01 63.5 0)
-		(effects
-			(font
-				(size 1.27 1.27)
-			)
-			(justify left)
-		)
-	)
-	(hierarchical_label "NRST"
-		(shape input)
-		(at 124.46 69.85 180)
-		(effects
-			(font
-				(size 1.27 1.27)
-			)
-			(justify right)
-		)
-	)
-	(hierarchical_label "JTDO-SWO"
-		(shape input)
-		(at 81.28 87.63 0)
 		(effects
 			(font
@@
 		)
 	)
-	(hierarchical_label "JTDO-SWO"
-		(shape input)
-		(at 124.46 64.77 180)
-		(effects
-			(font
-				(size 1.27 1.27)
-			)
-			(justify right)
-		)
-	)

Commit message: Updated files
Parts:
- TP2: footprint TestPoint:TestPoint_Pad_D2.0mm -> TestPoint:TestPoint_Loop_D2.60mm_Drill1.6mm_Beaded
Changed lines of the file:
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@@
 			)
 		)
-		(property "Footprint" "TestPoint:TestPoint_Pad_D2.0mm"
+		(property "Footprint" "TestPoint:TestPoint_Loop_D2.60mm_Drill1.6mm_Beaded"
 			(at 49.53 58.42 0)
 			(hide yes)

Commit message: Update
Parts:
- added C19: 0.1u, SCRB_STD_Passives:C0805, symbol SCRB_STD_Passives:C0805
- added J8: Conn_01x03, Connector_Hirose:Hirose_DF57H-3P-1.2V_1x03_P1.2mm_Socket, symbol Connector_Generic:Conn_01x03
- added R22: 120, SCRB_STD_Passives:R0805, symbol SCRB_STD_Passives:R0805
- added R44: 10k, SCRB_STD_Passives:R0805, symbol SCRB_STD_Passives:R0805
- added U11: THVD1500DR, SCRB_TexasInstruments:D0008A, symbol SCRB_TexasInstruments:THVD1500_D
- J6: KiLib_Generator (none) -> connector/SMD_single_row_plus_mounting_pad
Connections:
- net GND: now also C19.2, J8.3 (Pin_3), R44.1, U11.5 (GND)
- net JTCK-SWCLK: now also U3.9 (NC), J8.1 (Pin_1), R22.2, U11.6 (A)
- net RS485A: now reaches U3.4 (D3)
- net RS485A: now also U3.7 (NC), J8.2 (Pin_2), R22.1, U11.7 (B)
- new net: R44.2, U11.2 (nRE), U11.3 (DE)
- new net 5V: C19.1, U11.8 (VCC)
- new net USART6_RX: U11.1 (R)
- new net USART6_TX: U11.4 (D)
- no-connect marks 6 -> 3
Other:
- note added: "MCU Comunication to Main Board"
- note added: "RS485 - URC board to Main Payload Board"
- note added: "UART transceiver"
- moved on the sheet: J6, TP2, U3
