File: Hardware/Payload URC/photo_diode_circuit.kicad_sch (KiCad schematic)
At the start: 10 parts, among them U5 ADS1115IDGS, U7 OPA381

Commit message: Testing github skill issue
Parts:
- C18: value 0.1uF -> 0.1u; Voltage Voltage -> 25V
- C19: value 2.7pF -> 2.7p; Voltage Voltage -> 25V
- R44: value 100kΩ -> 100k
- R45: value 6.6kΩ -> 6.6k
Changed lines of the file:
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@@
 			)
 		)
-		(property "Value" "6.6kΩ"
+		(property "Value" "6.6k"
 			(at 39.37 115.5699 0)
 			(show_name no)
@@
 			)
 		)
-		(property "Value" "0.1uF"
+		(property "Value" "0.1u"
 			(at 123.19 64.3115 0)
 			(show_name no)
@@
 			)
 		)
-		(property "Voltage" "Voltage"
+		(property "Voltage" "25V"
 			(at 123.19 66.8515 0)
 			(show_name no)
@@
 			)
 		)
-		(property "Value" "2.7pF"
+		(property "Value" "2.7p"
 			(at 48.006 53.34 90)
 			(show_name no)
@@
 			)
 		)
-		(property "Voltage" "Voltage"
+		(property "Voltage" "25V"
 			(at 48.006 55.88 90)
 			(show_name no)
@@
 			)
 		)
-		(property "Value" "100kΩ"
+		(property "Value" "100k"
 			(at 50.8 68.58 90)
 			(show_name no)

Commit message: Updated files
Parts:
- removed C19: 2.7p, SCRB_STD_Passives:C0805, symbol SCRB_STD_Passives:C0805
- removed D4: BPW34, OptoDevice:Osram_DIL2_4.3x4.65mm_P5.08mm, symbol Sensor_Optical:BPW34
- removed R44: 100k, SCRB_STD_Passives:R0805, symbol SCRB_STD_Passives:R0805
- removed R45: 6.6k, SCRB_STD_Passives:R0805, symbol SCRB_STD_Passives:R0805
- removed TP24, TP26: TestPoint, TestPoint:TestPoint_Pad_D2.0mm, symbol Connector:TestPoint
- removed U7: OPA381, Package_TO_SOT_SMD:SOT-23-5, symbol Amplifier_Operational:LM321
- added J9: Conn_01x03, Connector_Hirose:Hirose_DF57H-3P-1.2V_1x03_P1.2mm_Socket, symbol Connector_Generic:Conn_01x03
- TP21: footprint TestPoint:TestPoint_Pad_D2.0mm -> TestPoint:TestPoint_Loop_D2.60mm_Drill1.6mm_Beaded
Connections:
- net GND: now also J9.3 (Pin_3)
- net at U5.5 (AIN1): now also J9.2 (Pin_2)
- net OPA381_AIN0: no longer names the net of TP21.1, U5.4 (AIN0)
- net OPA381_AIN0: now also J9.1 (Pin_1)
- no-connect marks 3 -> 2
Other:
- note added: "C2 calculations The purpose of C2 is to constrain the bandwidth to 18MHz OPA381's datasheet gives 2 formulas for C2: 2. 1/(2π * Rf * (Cf + C STRAY) = square root of [ (GBW/4π* Rf * CTOT) ] 2. CTOT = CDiode + 2.5 pF + 1 pF Given values from datasheet: 1. CTOT = 40 pF + 2.5 pF + 1 pF = 43.5 pF 2. C STRAY = 0.2 pF 3. GBW of OPA381= 18MHz Rf=1 000 000 ohms Plugging all of these into the above formula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"
- note removed: "0.35mV"
- note removed: "C2 calculations The purpose of C2 is to constrain the bandwidth to 18MHz OPA381's datasheet gives 2 formulas for C2: 2. 1/(2π * Rf * (Cf + C STRAY) = square root of [ (GBW/4π* Rf * CTOT) ] 2. CTOT = CDiode + 2.5 pF + 1 pF Given values from datasheet: 1. CTOT = 40 pF + 2.5 pF + 1 pF = 43.5 pF 2. C STRAY = 0.2 pF 3. GBW of OPA381= 18MHz Rf=100k ohms Plugging all of these into the above formula and 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"
- note removed: "Photo diode + OP-AMP circuit"
- note removed: "Photodiode's R44 will be a placeholder. Determined at component testing."
- note removed: "Simulation results indicate that the voltage at the output of the photodiode circuit is 0.35 mV."
- moved on the sheet: C18, TP21, U5

Commit message: Update
Parts:
- U5: KiLib_Generator (none) -> package/gullwing
Changed lines of the file:
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@@
+			)
+		)
+		(property "KiLib_Generator" "package/gullwing"
+			(at 196.85 101.6 0)
+			(hide yes)
+			(show_name no)
+			(do_not_autoplace no)
+			(effects
+				(font
+					(size 1.27 1.27)
+				)
 			)
 		)
