File: Hardware/Payload URC/solenoids.kicad_sch (KiCad schematic)
At the start: 14 parts, among them J2 Conn_01x02, J3 Conn_01x02, Q5 AO3400A, Q6 AO3400A

Commit message: Testing github skill issue
Parts:
- J2, J3: footprint Connector_JST:JST_XH_B2B-XH-A_1x02_P2.50mm_Vertical -> SCRB_Connectors:JST-GH-SM04B-GHS-TB
- R24, R33, R36, R37: value 100Ω -> 100
- R34, R35: value 10kΩ -> 10k
Changed lines of the file:
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@@
 			)
 		)
-		(property "Footprint" "Connector_JST:JST_XH_B2B-XH-A_1x02_P2.50mm_Vertical"
+		(property "Footprint" "SCRB_Connectors:JST-GH-SM04B-GHS-TB"
 			(at 132.08 44.45 0)
 			(hide yes)
@@
 			)
 		)
-		(property "Value" "100Ω"
+		(property "Value" "100"
 			(at 109.22 55.88 90)
 			(show_name no)
@@
 			)
 		)
-		(property "Value" "10kΩ"
+		(property "Value" "10k"
 			(at 46.99 69.8499 0)
 			(show_name no)
@@
 			)
 		)
-		(property "Footprint" "Connector_JST:JST_XH_B2B-XH-A_1x02_P2.50mm_Vertical"
+		(property "Footprint" "SCRB_Connectors:JST-GH-SM04B-GHS-TB"
 			(at 63.5 48.26 0)
 			(hide yes)
@@
 			)
 		)
-		(property "Value" "100Ω"
+		(property "Value" "100"
 			(at 39.37 58.42 90)
 			(show_name no)
@@
 			)
 		)
-		(property "Value" "10kΩ"
+		(property "Value" "10k"
 			(at 115.57 67.3099 0)
 			(show_name no)
@@
 			)
 		)
-		(property "Value" "100Ω"
+		(property "Value" "100"
 			(at 125.73 30.4799 0)
 			(show_name no)
@@
 			)
 		)
-		(property "Value" "100Ω"
+		(property "Value" "100"
 			(at 57.15 33.0199 0)
 			(show_name no)

Commit message: Updated files
Parts:
- J2, J3: footprint SCRB_Connectors:JST-GH-SM04B-GHS-TB -> Connector_JST:JST_PH_S2B-PH-K_1x02_P2.00mm_Horizontal
- TP14, TP16: footprint TestPoint:TestPoint_Pad_D2.0mm -> TestPoint:TestPoint_Loop_D2.60mm_Drill1.6mm_Beaded
Changed lines of the file:
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@@
 			)
 		)
-		(property "Footprint" "SCRB_Connectors:JST-GH-SM04B-GHS-TB"
+		(property "Footprint" "Connector_JST:JST_PH_S2B-PH-K_1x02_P2.00mm_Horizontal"
 			(at 132.08 44.45 0)
 			(hide yes)
@@
 			)
 		)
-		(property "Footprint" "SCRB_Connectors:JST-GH-SM04B-GHS-TB"
+		(property "Footprint" "Connector_JST:JST_PH_S2B-PH-K_1x02_P2.00mm_Horizontal"
 			(at 63.5 48.26 0)
 			(hide yes)
@@
 			)
 		)
-		(property "Footprint" "TestPoint:TestPoint_Pad_D2.0mm"
+		(property "Footprint" "TestPoint:TestPoint_Loop_D2.60mm_Drill1.6mm_Beaded"
 			(at 95.25 62.23 0)
 			(hide yes)
@@
 			)
 		)
-		(property "Footprint" "TestPoint:TestPoint_Pad_D2.0mm"
+		(property "Footprint" "TestPoint:TestPoint_Loop_D2.60mm_Drill1.6mm_Beaded"
 			(at 22.86 64.77 0)
 			(hide yes)

Commit message: Update
Parts:
- D8, D9: KiLib_Generator (none) -> diode/THT
- J2, J3: KiLib_Generator (none) -> connector/JST
- Q5, Q6: KiLib_Generator (none) -> package/gullwing
Changed lines of the file:
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@@
+			)
+		)
+		(property "KiLib_Generator" "connector/JST"
+			(at 132.08 44.45 0)
+			(hide yes)
+			(show_name no)
+			(do_not_autoplace no)
+			(effects
+				(font
+					(size 1.27 1.27)
+				)
 			)
 		)
@@
 			)
 		)
+		(property "KiLib_Generator" "diode/THT"
+			(at 140.97 45.72 0)
+			(hide yes)
+			(show_name no)
+			(do_not_autoplace no)
+			(effects
+				(font
+					(size 1.27 1.27)
+				)
+			)
+		)
 		(pin "1"
 		)
@@
 			)
 		)
+		(property "KiLib_Generator" "diode/THT"
+			(at 72.39 49.53 0)
+			(hide yes)
+			(show_name no)
+			(do_not_autoplace no)
+			(effects
+				(font
+					(size 1.27 1.27)
+				)
+			)
+		)
 		(pin "1"
 		)
@@
 			)
 		)
+		(property "KiLib_Generator" "connector/JST"
+			(at 63.5 48.26 0)
+			(hide yes)
+			(show_name no)
+			(do_not_autoplace no)
+			(effects
+				(font
+					(size 1.27 1.27)
+				)
+			)
+		)
 		(pin "2"
 		)
@@
 			)
 		)
+		(property "KiLib_Generator" "package/gullwing"
+			(at 52.07 64.77 0)
+			(hide yes)
+			(show_name no)
+			(do_not_autoplace no)
+			(effects
+				(font
+					(size 1.27 1.27)
+				)
+			)
+		)
 		(pin "3"
 		)
@@
 			(at 120.65 62.23 0)
 			(hide yes)
+			(show_name no)
+			(do_not_autoplace no)
+			(effects
+				(font
+					(size 1.27 1.27)
+				)
+			)
+		)
+		(property "KiLib_Generator" "package/gullwing"
+			(at 120.65 62.23 0)
+			(hide yes)
