File: Hardware/Payload URC/ultrasonic_vibrator.kicad_sch (KiCad schematic)
At the start: 7 parts, among them J1 VG2080001H, U2 DRV2605LDGS

Commit message: Testing github skill issue
Parts:
- C20, C21: value 1uF -> 1u; Voltage Voltage -> 25V
- J1: footprint Connector_JST:JST_XH_B2B-XH-A_1x02_P2.50mm_Vertical -> SCRB_Connectors:JST-GH-SM04B-GHS-TB
Changed lines of the file:
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@@
 			)
 		)
-		(property "Value" "1uF"
+		(property "Value" "1u"
 			(at 96.52 69.85 90)
 			(show_name no)
@@
 			)
 		)
-		(property "Voltage" "Voltage"
+		(property "Voltage" "25V"
 			(at 96.52 67.31 90)
 			(show_name no)
@@
 			)
 		)
-		(property "Value" "1uF"
+		(property "Value" "1u"
 			(at 92.71 30.48 90)
 			(show_name no)
@@
 			)
 		)
-		(property "Voltage" "Voltage"
+		(property "Voltage" "25V"
 			(at 92.71 33.02 90)
 			(show_name no)
@@
 			)
 		)
-		(property "Footprint" "Connector_JST:JST_XH_B2B-XH-A_1x02_P2.50mm_Vertical"
+		(property "Footprint" "SCRB_Connectors:JST-GH-SM04B-GHS-TB"
 			(at 168.91 49.53 0)
 			(hide yes)

Commit message: Updated files
Parts:
- TP35, TP36, TP37: footprint TestPoint:TestPoint_Pad_D2.0mm -> TestPoint:TestPoint_Loop_D2.60mm_Drill1.6mm_Beaded
Changed lines of the file:
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@@
 			)
 		)
-		(property "Footprint" "TestPoint:TestPoint_Pad_D2.0mm"
+		(property "Footprint" "TestPoint:TestPoint_Loop_D2.60mm_Drill1.6mm_Beaded"
 			(at 38.1 52.07 0)
 			(hide yes)
@@
 			)
 		)
-		(property "Footprint" "TestPoint:TestPoint_Pad_D2.0mm"
+		(property "Footprint" "TestPoint:TestPoint_Loop_D2.60mm_Drill1.6mm_Beaded"
 			(at 38.1 68.58 0)
 			(hide yes)
@@
 			)
 		)
-		(property "Footprint" "TestPoint:TestPoint_Pad_D2.0mm"
+		(property "Footprint" "TestPoint:TestPoint_Loop_D2.60mm_Drill1.6mm_Beaded"
 			(at 38.1 58.42 0)
 			(hide yes)

Commit message: Update
Parts:
- removed TP36, TP37: TestPoint, TestPoint:TestPoint_Loop_D2.60mm_Drill1.6mm_Beaded, symbol Connector:TestPoint
- removed U2: DRV2605LDGS, Package_SO:VSSOP-10_3x3mm_P0.5mm, symbol Driver_Haptic:DRV2605LDGS
- added U1: DRV2605LDGS, Package_SO:TSSOP-10_3x3mm_P0.5mm, symbol Driver:DRV2605LDGS
Connections:
- net 3V3: now also U1.10 (VDD)
- net GND: now also U1.4 (IN/TRIG), U1.8 (GND)
- net GPIO1: now also U1.5 (EN)
- net I2C1_SCL: now also U1.2 (SCL)
- net I2C1_SDA: now also U1.3 (SDA)
- net at C21.1: now also U1.1 (REG)
- net at J1.1 (Pin_1): now also U1.7 (OUT+)
- net at J1.2 (Pin_2): now also U1.9 (OUT-)
